File: Eagle/2_Out_Headphone_Amp.sch (EAGLE design)
At the start: 1 part, among them IC1 OPA2134P

Commit message: ヘッドホンアンプの修正
Parts:
- added C1, C9: 1.0u, rcl:C-EU050-045X075
- added C10, C5, C6, C7, C8: 0.1u, rcl:C-EU050-024X044
- added C11, C2: (no value), rcl:CPOL-EUTT5D11L
- added C4: 0.i1, rcl:C-EU050-024X044
- added IC2, IC3: OPA2134P, burr-brown:OPA2134P
- added JP1: IN-L, pinhead:PINHD-1X2
- added JP2: (no value), pinhead:PINHD-1X2
- added JP3: +3V, pinhead:PINHD-1X2
- added JP4: -3V, pinhead:PINHD-1X2
- added JP5: OUT1, pinhead:PINHD-1X3
- added JP6: OUT2, pinhead:PINHD-1X3
- added R1, R6: 100k, rcl:R-EU_0207/7
- added R10, R2, R5, R9: 47, rcl:R-EU_0207/7
- added R3, R7: 2k, rcl:R-EU_0207/7
- added R4, R8: 1k, rcl:R-EU_0207/7
Connections:
- new net +3V: C11.+, C4.2, C6.2, C8.2, JP3.2
- new net -3V: C10.1, C2.-, C5.1, C7.1, JP4.1
- new net GND: C10.2, C11.-, C2.+, C4.1, C5.2, C6.1, C7.2, C8.1, JP1.2, JP2.2, JP3.1, JP4.2, JP5.2, JP6.2, R1.1, R4.1, R6.1, R8.1
- new net N$10: C9.2, IC1B.+IN, R6.2
- new net N$11: IC1B.-IN, R7.1, R8.2
- new net N$12: IC1B.OUT, IC2B.+IN, IC3B.+IN, R7.2
- new net N$13: IC2B.-IN, IC2B.OUT, R9.1
- new net N$14: IC3B.-IN, IC3B.OUT, R10.1
- new net N$15: JP5.3, R9.2
- new net N$16: JP6.3, R10.2
- new net N$4: IC1A.OUT, IC2A.+IN, IC3A.+IN, R3.2
- new net N$5: IC2A.-IN, IC2A.OUT, R2.1
- new net N$6: JP5.1, R2.2
- new net N$7: IC3A.-IN, IC3A.OUT, R5.1
- new net N$8: JP6.1, R5.2
- new net N$9: C9.1, JP2.1
- new net V+: IC1A.V+, IC2A.V+, IC3A.V+
- new net V-: IC1A.V-, IC2A.V-, IC3A.V-
- net N$1: now also C1.1, JP1.1; no longer IC1A.-IN, IC1B.-IN
- net N$2: now also C1.2, R1.2; no longer IC1B.+IN
- net N$3: now also IC1A.-IN, R3.1, R4.2; no longer IC1A.OUT, IC1B.OUT
Other:
- moved on the sheet: IC1A, IC1B

Commit message: 回路図修正
Parts:
- JP2: value (none) -> IN-R
Changed lines of the file:
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@@
 <setting verticaltext="up"/>
 </settings>
-<grid distance="0.1" unitdist="inch" unit="inch" style="dots" multiple="1" display="yes" altdistance="0.01" altunitdist="inch" altunit="inch"/>
+<grid distance="0.1" unitdist="inch" unit="inch" style="lines" multiple="1" display="no" altdistance="0.01" altunitdist="inch" altunit="inch"/>
 <layers>
 <layer number="1" name="Top" color="4" fill="1" visible="no" active="no"/>
@@
 <part name="IC3" library="burr-brown" deviceset="OPA2134" device="P"/>
 <part name="JP1" library="pinhead" deviceset="PINHD-1X2" device="" value="IN-L"/>
-<part name="JP2" library="pinhead" deviceset="PINHD-1X2" device=""/>
+<part name="JP2" library="pinhead" deviceset="PINHD-1X2" device="" value="IN-R"/>
 <part name="C1" library="rcl" deviceset="C-EU" device="050-045X075" value="1.0u"/>
 <part name="R1" library="rcl" deviceset="R-EU_" device="0207/7" value="100k"/>

Commit message: 基板設計図追加
Parts:
- C11, C2: value (none) -> 1000u
Connections:
- removed net +3V: C11.+, C4.2, C6.2, C8.2, JP3.2
- removed net -3V: C10.1, C2.-, C5.1, C7.1, JP4.1
- net V+: now also C11.+, C4.2, C6.2, C8.2, JP3.2
- net V-: now also C10.1, C2.-, C5.1, C7.1, JP4.1
Other:
- moved on the sheet: C10, C11, C2, C4, C5, C6, C7, C8

Commit message: 基板設計図の変更
Parts:
- R1, R4, R6, R7, R8: device rcl:R-EU_0207/7 -> rcl:R-EU_0207/2V
Changed lines of the file:
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@@
 <part name="JP2" library="pinhead" deviceset="PINHD-1X2" device="" value="IN-R"/>
 <part name="C1" library="rcl" deviceset="C-EU" device="050-045X075" value="1.0u"/>
-<part name="R1" library="rcl" deviceset="R-EU_" device="0207/7" value="100k"/>
+<part name="R1" library="rcl" deviceset="R-EU_" device="0207/2V" value="100k"/>
 <part name="R2" library="rcl" deviceset="R-EU_" device="0207/7" value="47"/>
 <part name="GND1" library="supply1" deviceset="GND" device=""/>
 <part name="R3" library="rcl" deviceset="R-EU_" device="0207/7" value="2k"/>
-<part name="R4" library="rcl" deviceset="R-EU_" device="0207/7" value="1k"/>
+<part name="R4" library="rcl" deviceset="R-EU_" device="0207/2V" value="1k"/>
 <part name="GND2" library="supply1" deviceset="GND" device=""/>
 <part name="R5" library="rcl" deviceset="R-EU_" device="0207/7" value="47"/>
@@
 <part name="C9" library="rcl" deviceset="C-EU" device="050-045X075" value="1.0u"/>
 <part name="GND6" library="supply1" deviceset="GND" device=""/>
-<part name="R6" library="rcl" deviceset="R-EU_" device="0207/7" value="100k"/>
+<part name="R6" library="rcl" deviceset="R-EU_" device="0207/2V" value="100k"/>
 <part name="GND7" library="supply1" deviceset="GND" device=""/>
 <part name="GND8" library="supply1" deviceset="GND" device=""/>
-<part name="R7" library="rcl" deviceset="R-EU_" device="0207/7" value="2k"/>
-<part name="R8" library="rcl" deviceset="R-EU_" device="0207/7" value="1k"/>
+<part name="R7" library="rcl" deviceset="R-EU_" device="0207/2V" value="2k"/>
+<part name="R8" library="rcl" deviceset="R-EU_" device="0207/2V" value="1k"/>
 <part name="R9" library="rcl" deviceset="R-EU_" device="0207/7" value="47"/>
 <part name="R10" library="rcl" deviceset="R-EU_" device="0207/7" value="47"/>
